File: Electronics/kicad/project_alpha/_autosave-Lab1.kicad_pcb (KiCad board)
At the start: 2 copper layers, 80 x 107 mm, 102 parts, among them J1 USB_OTG, J2 USB_B_Micro, J3 Conn_01x03_Female, J4 Conn_01x06_Female, J5 Conn_01x06_Female, SW1 SW_Push, SW2 SW_Push, SW3 SW_Push, SW4 SW_Push, SW5 SW_Push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

Commit message: begin designing PCB
Parts:
- C15: footprint Capacitor_SMD:C_Elec_6.3x7.7 -> Capacitor_SMD:CP_Elec_4x5.4
- C20, C21, C37, C38, C39, C40, C41: footprint Capacitor_SMD:CP_Elec_5x5.9 -> Capacitor_SMD:CP_Elec_4x5.4
- C28, C29: footprint Capacitor_SMD:C_Elec_6.3x7.7 -> Capacitor_SMD:C_0805_2012Metric_Pad1.15x1.40mm_HandSolder
- moved H1 187.4 mm to (139.7, 61.0)
- moved C5 184.5 mm to (114.7, 93.2), turned to 270 degrees
- moved C13 171.7 mm to (126.5, 101.0)
- moved C20 163.3 mm to (137.2, 88.9), turned to 270 degrees
- moved C38 159.7 mm to (163.0, 83.1), turned to 270 degrees
- moved C11 146.1 mm to (141.0, 82.5), turned to 270 degrees
- moved SW3 145.6 mm to (116.5, 111.1), turned to 180 degrees
- moved C9 141.3 mm to (121.7, 89.2), turned to 270 degrees
- moved R14 141.3 mm to (165.0, 98.0)
- moved C29 140.2 mm to (158.0, 82.8), turned to 270 degrees
- moved R13 139.0 mm to (165.0, 96.0)
- moved SW4 135.1 mm to (127.5, 111.1), turned to 180 degrees
- moved C23 131.9 mm to (146.5, 75.2), turned to 270 degrees
- moved SW1 125.1 mm to (138.5, 111.1), turned to 180 degrees
- moved C28 125.0 mm to (146.1, 83.6), turned to 90 degrees
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Connections:
- C29 pad 2: GNDA -> GNDD
- C38 pad 2: GNDA -> GNDD
Routing:
- net /USB_ID: track 0.00 -> 35.9 mm
- net Net-(J2-Pad3): track 0.00 -> 23.6 mm
- net Net-(J2-Pad2): track 0.00 -> 23.6 mm
- net /USB_DP: track 0.00 -> 6.97 mm
- net /USB_DM: track 0.00 -> 6.35 mm
