File: Electronics/kicad/project_alpha/Buttons.sch (KiCad schematic (older format))
At the start: 20 parts, among them SW1 SW_Push, SW2 SW_Push, SW3 SW_Push, SW4 SW_Push, SW5 SW_Push

Commit message: finnished PCB routeing, added gerber files
Parts:
- C19, C33, C35, C36, C42: value 0.1u -> 100n
Changed lines of the file:
@@
 AR Path="/5C725C26/5C74F401" Ref="C33"  Part="1"
 F 0 "C33" H 1515 4296 50  0000 L CNN
-F 1 "0.1u" H 1515 4205 50  0000 L CNN
+F 1 "100n" H 1515 4205 50  0000 L CNN
 F 2 "Capacitor_SMD:C_0805_2012Metric_Pad1.15x1.40mm_HandSolder" H 1438 4100 50  0001 C CNN
 F 3 "~" H 1400 4250 50  0001 C CNN
@@
 AR Path="/5C725C26/5C74F43B" Ref="C35"  Part="1"
 F 0 "C35" H 2765 4246 50  0000 L CNN
-F 1 "0.1u" H 2765 4155 50  0000 L CNN
+F 1 "100n" H 2765 4155 50  0000 L CNN
 F 2 "Capacitor_SMD:C_0805_2012Metric_Pad1.15x1.40mm_HandSolder" H 2688 4050 50  0001 C CNN
 F 3 "~" H 2650 4200 50  0001 C CNN
@@
 AR Path="/5C725C26/5C74F475" Ref="C36"  Part="1"
 F 0 "C36" H 4065 4196 50  0000 L CNN
-F 1 "0.1u" H 4065 4105 50  0000 L CNN
+F 1 "100n" H 4065 4105 50  0000 L CNN
 F 2 "Capacitor_SMD:C_0805_2012Metric_Pad1.15x1.40mm_HandSolder" H 3988 4000 50  0001 C CNN
 F 3 "~" H 3950 4150 50  0001 C CNN
@@
 AR Path="/5C725C26/5C797646" Ref="C42"  Part="1"
 F 0 "C42" H 6615 4246 50  0000 L CNN
-F 1 "0.1u" H 6615 4155 50  0000 L CNN
+F 1 "100n" H 6615 4155 50  0000 L CNN
 F 2 "Capacitor_SMD:C_0805_2012Metric_Pad1.15x1.40mm_HandSolder" H 6538 4050 50  0001 C CNN
 F 3 "~" H 6500 4200 50  0001 C CNN
@@
 AR Path="/5C725C26/5C79767F" Ref="C19"  Part="1"
 F 0 "C19" H 5365 4196 50  0000 L CNN
-F 1 "0.1u" H 5365 4105 50  0000 L CNN
+F 1 "100n" H 5365 4105 50  0000 L CNN
 F 2 "Capacitor_SMD:C_0805_2012Metric_Pad1.15x1.40mm_HandSolder" H 5288 4000 50  0001 C CNN
 F 3 "~" H 5250 4150 50  0001 C CNN
