File: Electronics/kicad/project_alpha/Lab1.kicad_pcb (KiCad board)
At the start: 2 copper layers, 80 x 107 mm, 102 parts, among them J1 USB_OTG, J2 USB_B_Micro, J3 Conn_01x03_Female, J4 Conn_01x06_Female, J5 Conn_01x06_Female, SW1 SW_Push, SW2 SW_Push, SW3 SW_Push, SW4 SW_Push, SW5 SW_Push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

Commit message: update PCB, not done yet
Parts:
- C15, C22: footprint Capacitor_SMD:C_Elec_6.3x7.7 -> Capacitor_SMD:CP_Elec_4x5.4
- C20, C21, C39, C40, C41: footprint Capacitor_SMD:CP_Elec_5x5.9 -> Capacitor_SMD:CP_Elec_4x5.4
- C23: value 47u -> 10u
- C28, C29: footprint Capacitor_SMD:C_Elec_6.3x7.7 -> Capacitor_SMD:C_0805_2012Metric_Pad1.15x1.40mm_HandSolder
- C37, C38: footprint Capacitor_SMD:CP_Elec_5x5.9 -> Capacitor_SMD:C_0805_2012Metric_Pad1.15x1.40mm_HandSolder
- moved R9 199.1 mm to (130.0, 59.5), turned to 270 degrees
- moved R3 194.9 mm to (112.0, 81.0), turned to 270 degrees
- moved C5 190.8 mm to (106.2, 65.6), turned to 180 degrees
- moved C30 188.0 mm to (124.5, 59.5), turned to 90 degrees
- moved R4 185.7 mm to (114.0, 81.0), turned to 270 degrees
- moved C27 183.2 mm to (119.0, 67.0), turned to 90 degrees
- moved C31 180.5 mm to (124.5, 68.0), turned to 90 degrees
- moved R11 177.0 mm to (133.5, 59.5), turned to 90 degrees
- moved R12 172.2 mm to (133.5, 64.5), turned to 90 degrees
- moved C13 168.5 mm to (128.5, 81.0), turned to 270 degrees
- moved C11 168.0 mm to (119.0, 81.2), turned to 270 degrees
- moved C38 165.1 mm to (159.0, 89.0), turned to 90 degrees
- moved R10 164.0 mm to (130.0, 64.5), turned to 270 degrees
- moved R6 161.0 mm to (160.0, 71.0)
- moved R5 158.6 mm to (168.0, 71.0)
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Connections:
- C22 pad 1: GNDA -> Net-(C22-Pad1)
- C22 pad 2: Net-(C22-Pad2) -> GNDA
- C24 pad 1: Net-(C22-Pad2) -> Net-(C22-Pad1)
- C29 pad 2: GNDA -> GNDD
- C37 pad 1: +5V -> GNDA
- C37 pad 2: GNDA -> +5V
- C38 pad 2: GNDA -> GNDD
- U3 pad 18: Net-(C22-Pad2) -> Net-(C22-Pad1)
Other:
- board size 80 x 107 mm -> 100 x 100 mm

Commit message: update PCB
Parts:
- removed R1: 10K, Resistor_SMD:R_0805_2012Metric_Pad1.15x1.40mm_HandSolder
- added C43: 0.1u, Capacitor_SMD:C_0805_2012Metric_Pad1.15x1.40mm_HandSolder, F.Cu at (115.0, 91.0)
- added SW6: SW_Push, Button_Switch_SMD:SW_SPST_B3S-1000, F.Cu at (107.0, 91.0)
- C23: footprint Capacitor_SMD:C_Elec_6.3x7.7 -> Capacitor_SMD:CP_Elec_5x5.4
- R22: moved to F.Cu
- moved C42 222.7 mm to (123.0, 140.0)
- moved R36 219.8 mm to (119.0, 141.5), turned to 270 degrees
- moved C36 211.0 mm to (135.0, 140.0)
- moved R17 210.9 mm to (104.0, 107.0)
- moved R34 202.8 mm to (123.0, 143.0)
- moved R24 201.1 mm to (147.0, 143.0)
- moved R30 189.3 mm to (131.0, 141.5), turned to 270 degrees
- moved SW4 187.8 mm to (321.0, 139.0), turned to 0 degrees
- moved R16 186.9 mm to (151.0, 115.0), turned to 270 degrees
- moved R26 181.0 mm to (135.0, 143.0)
- moved C22 173.9 mm to (139.0, 84.8), turned to 90 degrees
- moved C25 171.9 mm to (144.0, 83.0)
- moved R2 165.0 mm to (147.0, 95.0), turned to 180 degrees
- moved C6 159.2 mm to (139.0, 101.0), turned to 180 degrees
- moved C35 158.7 mm to (147.0, 140.0)
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Connections:
- C10 pad 2: GNDD -> GNDA
- J2 pad 5: GNDA -> GNDD
- J2 pad 6: GNDA -> GNDD
- R2 pad 2: GND -> GNDD

Commit message: update PCB
Parts:
- removed R36: 1k, Resistor_SMD:R_0805_2012Metric_Pad1.15x1.40mm_HandSolder
- added R1: 10k, Resistor_SMD:R_0805_2012Metric_Pad1.15x1.40mm_HandSolder, F.Cu at (179.0, 65.5)
- C15: footprint Capacitor_SMD:CP_Elec_4x5.4 -> Capacitor_SMD:C_0805_2012Metric_Pad1.15x1.40mm_HandSolder
- R22, R24, R26, R35: value 10k -> 1k
- R23, R25, R30: value 1k -> 10k
- moved R18 252.1 mm to (120.0, 126.0), turned to 270 degrees
- moved D1 242.4 mm to (119.0, 132.1)
- moved D3 236.0 mm to (131.0, 132.1)
- moved R20 232.6 mm to (132.0, 126.5), turned to 270 degrees
- moved D2 230.9 mm to (125.0, 132.1)
- moved D4 216.8 mm to (137.0, 132.1)
- moved H1 212.2 mm to (113.5, 72.0)
- moved R19 211.0 mm to (126.4, 126.5), turned to 270 degrees
- moved R23 198.2 mm to (124.0, 144.0)
- moved C15 193.7 mm to (141.0, 114.9), turned to 90 degrees
- moved C33 192.6 mm to (124.0, 141.0)
- moved R33 192.3 mm to (144.5, 142.5), turned to 270 degrees
- moved R21 182.1 mm to (138.0, 126.5), turned to 270 degrees
- moved SW4 162.7 mm to (179.0, 59.5), turned to 180 degrees
- moved R22 152.6 mm to (174.5, 66.5), turned to 90 degrees
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Connections:
- C19 pad 1: /Button5 -> /Button4
- C33 pad 1: /Button4 -> /Button1
- C33 pad 2: GNDD -> GNDA
- C35 pad 1: /Button1 -> /Button2
- C35 pad 2: GNDD -> GNDA
- C36 pad 1: /Button2 -> /Button3
- C36 pad 2: GNDD -> GNDA
- C42 pad 1: /Button3 -> /Button5
- R22 pad 1: Net-(R22-Pad1) -> /Button4
- R22 pad 2: GNDD -> Net-(R1-Pad1)
- R23 pad 1: /Button4 -> Net-(R23-Pad1)
- R23 pad 2: Net-(R22-Pad1) -> GNDA
- R24 pad 1: Net-(R24-Pad1) -> /Button1
- R24 pad 2: GNDD -> Net-(R23-Pad1)
- R25 pad 1: /Button1 -> Net-(R25-Pad1)
- R25 pad 2: Net-(R24-Pad1) -> GNDA
- R26 pad 1: Net-(R26-Pad1) -> /Button2
- R26 pad 2: GNDD -> Net-(R25-Pad1)
- R30 pad 1: /Button2 -> Net-(R30-Pad1)
- R30 pad 2: Net-(R26-Pad1) -> GNDA
- R31 pad 2: /SPI_MOSI -> /LCD_SPI_MOSI
- R32 pad 2: /SPI_MISO -> /LCD_SPI_MISO
- R33 pad 1: /Button5 -> /Button3
- R33 pad 2: Net-(R33-Pad2) -> Net-(R30-Pad1)
- R35 pad 1: Net-(R33-Pad2) -> /Button5
- R35 pad 2: GNDD -> Net-(R34-Pad1)
- SW1 pad 1: Net-(R22-Pad1) -> Net-(R23-Pad1)
- SW2 pad 1: Net-(R24-Pad1) -> Net-(R25-Pad1)
- SW3 pad 1: Net-(R26-Pad1) -> Net-(R30-Pad1)
- SW4 pad 1: Net-(R33-Pad2) -> Net-(R1-Pad1)
- U4 pad 24: /SPI_MOSI -> /LCD_SPI_MOSI
- U4 pad 25: /SPI_SCK -> /LCD_SPI_SCK
- U4 pad 26: /SPI_MISO -> /LCD_SPI_MISO

Commit message: started routing PCB
Parts:
- moved C1 5.02 mm to (155.4, 120.6)
- moved C15 5.02 mm to (141.5, 119.9)
- moved C16 5.02 mm to (144.6, 119.9)
- moved C3 5.02 mm to (155.3, 123.6)
- moved R15 5.02 mm to (148.5, 120.0)
- moved R16 5.02 mm to (151.5, 120.0)
- moved C10 3.50 mm to (139.5, 104.0)
- moved C2 3.50 mm to (138.5, 110.0)
- moved C6 3.50 mm to (135.5, 101.0)
- moved C7 3.50 mm to (135.5, 107.0)
- moved Y1 3.50 mm to (130.5, 104.0)
- moved C17 3.00 mm to (159.0, 104.0)
- moved C4 3.00 mm to (147.0, 101.0)
- moved R2 3.00 mm to (147.0, 98.0)
- moved R29 3.00 mm to (154.0, 101.0)
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Routing:
- net GNDA: track 0.00 -> 50.4 mm
- net +5V: track 0.00 -> 22.5 mm
- net Net-(R3-Pad2): track 0.00 -> 13.5 mm
- net +3V3: track 0.00 -> 11.4 mm
Other:
- net class Power: trace_width 0.25 -> 0.4
- rule via_min_size: 0.4 -> 0.3

Commit message: finnished PCB routeing, added gerber files
Parts:
- added C44: 100p, Capacitor_SMD:C_0805_2012Metric_Pad1.15x1.40mm_HandSolder, F.Cu at (117.5, 60.0)
- added C45: 100p, Capacitor_SMD:C_0805_2012Metric_Pad1.15x1.40mm_HandSolder, F.Cu at (117.0, 66.0)
- C19, C24, C25, C28, C29, C33, C34, C35, C36, C42, C43: value 0.1u -> 100n
- C22: footprint Capacitor_SMD:CP_Elec_4x5.4 -> Capacitor_SMD:CP_Elec_5x5.4
- C23: footprint Capacitor_SMD:CP_Elec_5x5.4 -> Capacitor_SMD:CP_Elec_4x5.3
- C26, C27: value 200p -> 100p
- C30, C31: footprint Capacitor_SMD:CP_Elec_5x5.9 -> Capacitor_SMD:CP_Elec_4x5.3
- C5: footprint Capacitor_SMD:CP_Elec_5x5.9 -> Capacitor_SMD:CP_Elec_4x5.4
- moved RV3 29.8 mm to (109.0, 122.2)
- moved J5 25.3 mm to (196.8, 85.0)
- moved C2 21.4 mm to (159.0, 103.7)
- moved C43 19.3 mm to (134.2, 92.7)
- moved SW6 19.3 mm to (126.2, 92.8)
- moved J2 15.5 mm to (204.7, 97.8), turned to 0 degrees
- moved RV1 15.0 mm to (109.0, 152.0)
- moved RV2 15.0 mm to (109.0, 137.0)
- moved R29 13.4 mm to (160.8, 112.5), turned to 90 degrees
- moved C10 11.1 mm to (142.0, 114.8), turned to 180 degrees
- moved R11 10.6 mm to (132.9, 70.1), turned to 0 degrees
- moved C30 9.75 mm to (124.7, 69.2), turned to 0 degrees
- moved C31 8.14 mm to (126.0, 60.0), turned to 0 degrees
- moved R9 7.70 mm to (132.9, 66.6), turned to 180 degrees
- moved C26 7.57 mm to (120.0, 68.0)
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Connections:
- U3 pad 12: /SPI_MOSI -> /CODEC_SPI_MOSI
- U4 pad 20: GNDA -> GNDD
- U4 pad 21: GNDA -> GNDD
Routing:
- net +3V3: track 11.4 -> 418.2 mm, vias 0 -> 6
- net GNDA: track 50.4 -> 411.3 mm, vias 0 -> 2
- net GNDD: track 0.00 -> 276.9 mm, vias 0 -> 3
- net +5V: track 22.5 -> 168.5 mm, vias 0 -> 5
- net /NRST: track 0.00 -> 142.2 mm, vias 0 -> 5
- net /Button3: track 0.00 -> 79.3 mm, vias 0 -> 2
- net /Button5: track 0.00 -> 73.6 mm
- net /Button2: track 0.00 -> 68.4 mm, vias 0 -> 2
- net /POT3: track 0.00 -> 66.5 mm, vias 0 -> 1
- net /SWCLK: track 0.00 -> 64.3 mm
- net /Button1: track 0.00 -> 61.1 mm, vias 0 -> 2
- net /POT2: track 0.00 -> 53.9 mm
- net /SWO: track 0.00 -> 53.0 mm
- net /Button4: track 0.00 -> 51.8 mm, vias 0 -> 2
- net Net-(R17-Pad2): track 0.00 -> 51.6 mm
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- added copper zone on B.Cu, net GNDA
- added copper zone on F.Cu, net GNDA
Other:
- net class Power: trace_width 0.4 -> 0.3

Commit message: updated PCB routeing and gerber files
Parts:
- added J6: Conn_01x02_Female, Connector_Molex:Molex_KK-254_AE-6410-02A_1x02_P2.54mm_Vertical, F.Cu at (122.0, 107.0)
- moved J3 9.00 mm to (161.9, 66.5), turned to 180 degrees
- moved C4 2.93 mm to (145.4, 98.5)
- moved R2 2.93 mm to (145.4, 95.5)
Connections:
- U2 pad 58: /CODEC_SPI_SCK -> /USART_TX
- U2 pad 59: /CODEC_SPI_MISO -> /USART_RX
- U2 pad 61: Net-(U2-Pad61) -> /CODEC_SPI_SCK
- U2 pad 62: Net-(U2-Pad62) -> /CODEC_SPI_MISO
Routing:
- net /USART_TX: track 0.00 -> 38.8 mm, vias 0 -> 1
- net /USART_RX: track 0.00 -> 36.6 mm, vias 0 -> 1
- net GNDA: track 411.3 -> 381.7 mm
- net GNDD: track 276.9 -> 291.4 mm
- net +3V3: track 418.2 -> 427.0 mm, vias 6 -> 8
- net Net-(C32-Pad2): track 17.0 -> 25.5 mm
- net Net-(R2-Pad1): track 5.80 -> 13.8 mm, vias 0 -> 2
- net Net-(C18-Pad1): track 17.9 -> 22.7 mm
- net /CODEC_SPI_SCK: track 41.9 -> 45.7 mm
- net /CODEC_SPI_MISO: track 42.4 -> 45.5 mm
- net +5V: track 168.5 -> 171.3 mm
- net /Button1: track 61.1 -> 63.8 mm
- net /Button2: track 68.4 -> 70.1 mm
- net /Button3: track 79.3 -> 80.9 mm
- net /CODEC_CS: track 39.5 -> 37.9 mm
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- added copper zone on F.Cu, net GNDD
Other:
- net class Default: trace_width 0.25 -> 0.3
- net class Power: trace_width 0.3 -> 0.5
- board text added: "TX RX"
